Commit message: cmd_vel working in gazebo

File: segway-master/segway_simulation/urdf/segway.URDF (robot description, URDF)
Before this commit: robot segway_simulation, 4 links, 3 joints
Links:
- link base_footprint: mass 1.0 -> 0.0
Joints:
- joint base_footprint_joint: origin xyz=0 0 0.025 rpy=-1.57 0 0 -> xyz=0 0 0.025 rpy=-1.57 0 -1.57
